Commit message: First working version

File: model/franka.urdf (robot description, URDF)
Before this commit: robot panda, 12 links, 11 joints
Links:
- added link world
- link panda_hand: mass None -> 0.73; geometry collision box size=0.055 0.04 0.198; visual mesh filename=visual/hand.dae
- link panda_leftfinger: mass None -> 0.015; geometry collision box size=0.03 0.005 0.047; collision box size=0.03 0.015 0.017
- link panda_link0: mass None -> 0.629769; geometry collision mesh filename=collision/link0.stl; visual mesh filename=visual/link0.dae
- link panda_link1: mass None -> 4.970684; geometry collision mesh filename=collision/link1.stl; visual mesh filename=visual/link1.dae
- link panda_link2: mass None -> 0.646926; geometry collision mesh filename=collision/link2.stl; visual mesh filename=visual/link2.dae
- link panda_link3: mass None -> 3.228604; geometry collision mesh filename=collision/link3.stl; visual mesh filename=visual/link3.dae
- link panda_link4: mass None -> 3.587895; geometry collision mesh filename=collision/link4.stl; visual mesh filename=visual/link4.dae
- link panda_link5: mass None -> 1.225946; geometry collision mesh filename=collision/link5.stl; visual mesh filename=visual/link5.dae
- link panda_link6: mass None -> 1.666555; geometry collision mesh filename=collision/link6.stl; visual mesh filename=visual/link6.dae
- link panda_link7: mass None -> 7.35522e-01; geometry collision mesh filename=collision/link7.stl; visual mesh filename=visual/link7.dae
- link panda_link8: geometry 
- link panda_rightfinger: mass None -> 0.015; geometry collision box size=0.03 0.005 0.047; collision box size=0.03 0.015 0.017
Joints:
- added joint world_joint: type fixed, parent world, child panda_link0, origin xyz=0 0 0 rpy=0 0 0
- joint panda_finger_joint2: mimic joint=panda_finger_joint1 -> (none)
- joint panda_joint1: limit lower=-2.8973 upper=2.8973 effort=87 velocity=2.1750 -> lower=-2.9671 upper=2.9671 effort=87 velocity=2.5
- joint panda_joint2: limit lower=-1.7628 upper=1.7628 effort=87 velocity=2.1750 -> lower=-1.8326 upper=1.8326 effort=87 velocity=2.5
- joint panda_joint3: limit lower=-2.8973 upper=2.8973 effort=87 velocity=2.1750 -> lower=-2.9671 upper=2.9671 effort=87 velocity=2.5
- joint panda_joint4: limit lower=-3.0718 upper=-0.0698 effort=87 velocity=2.1750 -> lower=-3.1416 upper=-0.4 effort=87 velocity=2.5
- joint panda_joint5: limit lower=-2.8973 upper=2.8973 effort=12 velocity=2.6100 -> lower=-2.9671 upper=2.9671 effort=12 velocity=3
- joint panda_joint6: limit lower=-0.0175 upper=3.7525 effort=12 velocity=2.6100 -> lower=-0.0873 upper=3.8223 effort=12 velocity=3
- joint panda_joint7: limit lower=-2.8973 upper=2.8973 effort=12 velocity=2.6100 -> lower=-2.9671 upper=2.9671 effort=12 velocity=3
- joint panda_joint8: axis (none) -> 0 0 0

Commit message: Calibrator first working

File: model/franka.urdf (robot description, URDF)
Before this commit: robot panda, 13 links, 12 joints
Links:
- link panda_link1: mass 4.970684 -> 4.97068
- link panda_link2: mass 0.646926 -> 0.646303
- link panda_link3: mass 3.228604 -> 3.22332
- link panda_link4: mass 3.587895 -> 3.57869
- link panda_link5: mass 1.225946 -> 1.21201
- link panda_link6: mass 1.666555 -> 1.65017
- link panda_link7: mass 7.35522e-01 -> 1.44666
