Commit message: Refactoring, second calibration, tests pass

File: model/franka_emulator/model.urdf (robot description, URDF)
Before this commit: robot panda, 13 links, 12 joints
Links:
- link panda_link1: mass 4.97068 -> 4.9706751871147938
- link panda_link2: mass 0.646303 -> 0.64712411452542207
- link panda_link3: mass 3.22332 -> 3.2283417206016849
- link panda_link4: mass 3.57869 -> 3.5877058164189872
- link panda_link5: mass 1.21201 -> 1.2258764841419181
- link panda_link6: mass 1.65017 -> 1.6660195957719575
- link panda_link7: mass 1.44666 -> 0.73598318978014388
